Commit message: urdf updates

File: src/gsim_urdf_pkg/urdf/gsim_urdf_pkg.urdf (robot description, URDF)
Before this commit: robot gsim_urdf_pkg, 6 links, 5 joints
Links:
- added link world
Joints:
- added joint base_to_world: type fixed, parent world, child base_link, origin xyz=0 0 0 rpy=0 0 0
- joint Joint_Fifth: limit lower=-0.1 upper=0.1 effort=10 velocity=2 -> lower=-0.1 upper=0.1 effort=20 velocity=0.5
- joint Joint_First: axis 0 0 0 -> 1 0 0; limit (none) -> lower=-0.1 upper=0.1 effort=20 velocity=0.5; origin xyz=-0.051662 -0.082969 0.05 rpy=0 0 0 -> xyz=-0.05 -0.08 0.05 rpy=0 0 0; type fixed -> prismatic
- joint Joint_Fourth: limit lower=-0.1 upper=0.1 effort=10 velocity=2 -> lower=-0.1 upper=0.1 effort=20 velocity=0.5
- joint Joint_Second: limit lower=-0.1 upper=0.1 effort=10 velocity=2 -> lower=-0.1 upper=0.1 effort=20 velocity=0.5
- joint Joint_Third: limit lower=-0.1 upper=0.1 effort=10 velocity=2 -> lower=-0.1 upper=0.1 effort=20 velocity=0.5

Commit message: updated urdf

File: src/gsim_urdf_pkg/urdf/gsim_urdf_pkg.urdf (robot description, URDF)
Before this commit: robot gsim_urdf_pkg, 7 links, 6 joints
Joints:
- joint Joint_Fifth: limit lower=-0.1 upper=0.1 effort=20 velocity=0.5 -> lower=-0.01 upper=0.01 effort=5 velocity=0.5
- joint Joint_First: limit lower=-0.1 upper=0.1 effort=20 velocity=0.5 -> lower=-0.01 upper=0.01 effort=5 velocity=0.5
- joint Joint_Fourth: limit lower=-0.1 upper=0.1 effort=20 velocity=0.5 -> lower=-0.01 upper=0.01 effort=5 velocity=0.5
- joint Joint_Second: limit lower=-0.1 upper=0.1 effort=20 velocity=0.5 -> lower=-0.01 upper=0.01 effort=5 velocity=0.5
- joint Joint_Third: limit lower=-0.1 upper=0.1 effort=20 velocity=0.5 -> lower=-0.01 upper=0.01 effort=5 velocity=0.5

Commit message: camera added  but

File: src/gsim_urdf_pkg/urdf/gsim_urdf_pkg.urdf (robot description, URDF)
Before this commit: robot gsim_urdf_pkg, 7 links, 6 joints
Links:
- added link camera_link, mass 0.1; collision box size=0.1 0.1 0.1; visual box size=0.1 0.1 0.1
Joints:
- added joint camera_joint: type fixed, parent base_link, child camera_link, origin xyz=1 0 1 rpy=0 0 0

Commit message: adjusted camera view in urdf file in gsim_urdf_pkg

File: src/gsim_urdf_pkg/urdf/gsim_urdf_pkg.urdf (robot description, URDF)
Before this commit: robot gsim_urdf_pkg, 8 links, 7 joints
Joints:
- joint camera_joint: origin xyz=1 0 1 rpy=0 0 0 -> xyz=-1 0 1 rpy=0 0 0

Commit message: updated urdf with some adjustments for change of movement from x to y-direction

File: src/gsim_urdf_pkg/urdf/gsim_urdf_pkg.urdf (robot description, URDF)
Before this commit: robot gsim_urdf_pkg, 8 links, 7 joints
Joints:
- joint Joint_Fifth: axis 1 0 0 -> 0 1 0
- joint Joint_First: axis 1 0 0 -> 0 1 0
- joint Joint_Fourth: axis 1 0 0 -> 0 1 0
- joint Joint_Second: axis 1 0 0 -> 0 1 0
- joint Joint_Third: axis 1 0 0 -> 0 1 0

Commit message: laserScan

File: src/gsim_urdf_pkg/urdf/gsim_urdf_pkg.urdf (robot description, URDF)
Before this commit: robot gsim_urdf_pkg, 8 links, 7 joints
Links:
- added link laser_link, mass 0.1; collision box size=0.05 0.05 0.05; visual box size=0.05 0.05 0.05
Joints:
- added joint laser_joint: type fixed, parent base_link, child laser_link, origin xyz=-1 0 0.1 rpy=0 0 0
